File: Project PCB Designs/LocIT.sch (EAGLE design)
At the start: 5 parts, among them J1 PRT-14017

Commit message: Add files via upload
Changed lines of the file:
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@@
 <part name="U$16" library="microbuilder" deviceset="VLIPO" device=""/>
 <part name="U$5" library="microbuilder" deviceset="GND" device=""/>
-<part name="U$6" library="microbuilder" deviceset="3.3V" device=""/>
 <part name="JP3" library="microbuilder" deviceset="HEADER-1X6" device="70MIL"/>
 <part name="U$7" library="microbuilder" deviceset="GND" device=""/>
-<part name="U$8" library="microbuilder" deviceset="3.3V" device=""/>
 <part name="JP5" library="microbuilder" deviceset="HEADER-1X9" device="70MIL"/>
 <part name="J1" library="PRT-14017" deviceset="PRT-14017" device=""/>
@@
 <attribute name="VALUE" x="204.216" y="203.2" size="1.27" layer="96"/>
 </instance>
-<instance part="U$6" gate="G$1" x="180.34" y="220.98" smashed="yes">
-<attribute name="VALUE" x="178.816" y="221.996" size="1.27" layer="96"/>
-</instance>
 <instance part="JP3" gate="A" x="198.12" y="205.74" smashed="yes">
 <attribute name="NAME" x="191.77" y="216.535" size="1.778" layer="95"/>
@@
 <instance part="U$7" gate="G$1" x="304.8" y="198.12" smashed="yes">
 <attribute name="VALUE" x="303.276" y="195.58" size="1.27" layer="96"/>
-</instance>
-<instance part="U$8" gate="G$1" x="279.4" y="213.36" smashed="yes">
-<attribute name="VALUE" x="277.876" y="214.376" size="1.27" layer="96"/>
 </instance>
 <instance part="JP5" gate="A" x="297.18" y="195.58" smashed="yes">
@@
 <wire x1="195.58" y1="210.82" x2="180.34" y2="210.82" width="0.1524" layer="91"/>
 <wire x1="180.34" y1="210.82" x2="180.34" y2="218.44" width="0.1524" layer="91"/>
-<pinref part="U$6" gate="G$1" pin="3.3V"/>
 <pinref part="JP3" gate="A" pin="2"/>
 </segment>
@@
 <wire x1="294.64" y1="203.2" x2="279.4" y2="203.2" width="0.1524" layer="91"/>
 <wire x1="279.4" y1="203.2" x2="279.4" y2="210.82" width="0.1524" layer="91"/>
-<pinref part="U$8" gate="G$1" pin="3.3V"/>
 <pinref part="JP5" gate="A" pin="2"/>
 </segment>

Commit message: Add files via upload
Parts:
- removed JP3: (no value), microbuilder:HEADER-1X670MIL
- added JP6, JP7: (no value), microbuilder:HEADER-1X670MIL
Connections:
- removed net !RESET_GPS: JP3.6
- removed net 3.3V_GPS: JP3.2
- removed net VCC_GPS: J1.2, JP3.1
- new net !RESET: JP6.6
- new net 1PPS: JP7.2
- new net N$1: J1.11, JP6.2
- new net RXI: JP7.4
- new net TXO: JP7.5
- new net VCC: JP6.1
- net GND: now also J1.40, JP6.3, JP7.1, JP7.6; no longer JP3.3
- net SCL: now also JP6.4; no longer JP3.4
- net SDA: now also JP6.5; no longer JP3.5
- net VCC1: now also J1.13; no longer J1.1
- net VCC_GYRO: now also J1.15; no longer J1.17
