File: Project PCB Designs/LocIT.brd (EAGLE design)
At the start: 55.5 x 57.1 mm, 5 parts, among them J1 PRT-14017

Commit message: Add files via upload
Other:
- board size 55.5 x 57.1 mm -> 51.7 x 57.1 mm
Changed lines of the file:
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@@
 <drawing>
 <settings>
-<setting alwaysvectorfont="yes"/>
+<setting alwaysvectorfont="no"/>
 <setting verticaltext="up"/>
 </settings>
@@
 <board>
 <plain>
-<wire x1="17.03604375" y1="20.32" x2="64.4948" y2="20.32" width="0" layer="20"/>
+<wire x1="20.84604375" y1="20.32" x2="64.4948" y2="20.32" width="0" layer="20"/>
 <wire x1="64.4948" y1="20.32" x2="68.25" y2="24.0752" width="0" layer="20" curve="90"/>
 <wire x1="68.25" y1="24.0752" x2="68.25" y2="73.720921875" width="0" layer="20"/>
 <wire x1="68.25" y1="73.720921875" x2="64.510921875" y2="77.46" width="0" layer="20" curve="90"/>
-<wire x1="64.510921875" y1="77.46" x2="17.018959375" y2="77.46" width="0" layer="20"/>
-<wire x1="17.018959375" y1="77.46" x2="12.7" y2="73.141040625" width="0" layer="20" curve="90"/>
-<wire x1="12.7" y1="73.141040625" x2="12.7" y2="24.65604375" width="0" layer="20"/>
-<wire x1="12.7" y1="24.65604375" x2="17.03604375" y2="20.32" width="0" layer="20" curve="90"/>
+<wire x1="64.510921875" y1="77.46" x2="20.828959375" y2="77.46" width="0" layer="20"/>
+<wire x1="20.828959375" y1="77.46" x2="16.51" y2="73.141040625" width="0" layer="20" curve="90"/>
+<wire x1="16.51" y1="73.141040625" x2="16.51" y2="24.65604375" width="0" layer="20"/>
+<wire x1="16.51" y1="24.65604375" x2="20.84604375" y2="20.32" width="0" layer="20" curve="90"/>
 <dimension x1="28.194" y1="21.59" x2="25.273" y2="46.99" x3="26.7335" y3="34.29" textsize="1.778" layer="47" dtype="horizontal" unit="inch"/>
 <text x="26.67" y="29.21" size="1.27" layer="21">SDA</text>

Commit message: Add files via upload
Parts:
- moved J1 22.9 mm to (26.7, 47.0)
- moved JP2 6.84 mm to (19.1, 34.3)
- moved JP4 5.24 mm to (66.0, 34.4)
Routing:
- net VCC_GPS: track 30.8 -> 7.96 mm
- net VCC_GYRO: track 29.9 -> 46.8 mm
- net GND: track 105.0 -> 114.8 mm
- net VCC1: track 43.9 -> 35.7 mm
- net SDA: track 77.1 -> 69.8 mm
- net SCL: track 76.2 -> 69.5 mm

Commit message: Add files via upload
Parts:
- moved J1 2.54 mm to (26.7, 49.5)
Routing:
- net VCC1: track 35.7 -> 42.6 mm
- net SDA: track 69.8 -> 76.6 mm
- net SCL: track 69.5 -> 74.0 mm
- net VCC_GPS: track 7.96 -> 8.98 mm

Commit message: Add files via upload
Parts:
- added JP7: (no value), microbuilder:1X06_ROUND_70
- renumbered JP3 to JP6
Connections:
- net !RESET_GPS renamed !RESET
- removed net 3.3V_GPS: JP6.2
- removed net VCC_GPS: J1.2, JP6.1
- new net 1PPS: JP7.2
- new net N$1: J1.11, JP6.2
- new net RXI: JP7.4
- new net TXO: JP7.5
- new net VCC: JP6.1
- net GND: now also J1.40, JP7.1, JP7.6
- net VCC1: now also J1.13; no longer J1.1
- net VCC_GYRO: now also J1.15; no longer J1.17
Routing:
- net GND: track 114.7 -> 162.0 mm
- net VCC1: track 42.6 -> 28.1 mm
- net N$1: track 0.00 -> 10.5 mm
- net VCC_GPS: track 8.98 -> 0.00 mm
- net SCL: track 74.0 -> 76.0 mm
- net VCC_GYRO: track 46.5 -> 48.1 mm
Changed lines of the file:
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@@
 <drawing>
 <settings>
-<setting alwaysvectorfont="yes"/>
+<setting alwaysvectorfont="no"/>
 <setting verticaltext="up"/>
 </settings>
@@
 <attribute name="VALUE" x="69.215" y="24.257" size="0.4064" layer="27" ratio="10" rot="R90"/>
 </element>
-<element name="JP3" library="microbuilder" package="1X06_ROUND_70" value="" x="19.05" y="60.96" smashed="yes" rot="R270">
-<attribute name="VALUE" x="17.145" y="68.58" size="0.4064" layer="27" ratio="10" rot="R270"/>
-</element>
 <element name="JP5" library="microbuilder" package="1X09_ROUND_70" value="" x="54.61" y="74.93" smashed="yes" rot="R180">
 <attribute name="VALUE" x="66.04" y="78.105" size="0.4064" layer="27" ratio="10" rot="R180"/>
@@
 <attribute name="SNAPEDA_LINK" value="https://www.snapeda.com/parts/PRT-14017/SparkFun+Electronics/view-part/?ref=snap" x="26.67" y="49.53" size="1.778" layer="28" rot="MR270" display="off"/>
 </element>
+<element name="JP6" library="microbuilder" package="1X06_ROUND_70" value="" x="19.05" y="60.96" smashed="yes" rot="R270">
+<attribute name="NAME" x="20.8788" y="68.6562" size="0.8128" layer="25" ratio="18" rot="R270"/>
+<attribute name="VALUE" x="17.145" y="68.58" size="0.4064" layer="27" ratio="10" rot="R270"/>
+</element>
+<element name="JP7" library="microbuilder" package="1X06_ROUND_70" value="" x="39.37" y="60.96" smashed="yes" rot="R270">
+<attribute name="NAME" x="41.1988" y="68.6562" size="0.8128" layer="25" ratio="18" rot="R270"/>
+<attribute name="VALUE" x="36.195" y="68.58" size="0.4064" layer="27" ratio="10" rot="R270"/>
+</element>
 </elements>
 <signals>
@@
 <contactref element="JP4" pad="7"/>
 <contactref element="JP4" pad="5"/>
-<contactref element="JP3" pad="3"/>
 <contactref element="JP5" pad="3"/>
 <wire x1="17.78" y1="39.37" x2="19.05" y2="38.1" width="0.4064" layer="16"/>
 <wire x1="17.78" y1="60.96" x2="17.78" y2="39.37" width="0.4064" layer="16"/>
-<wire x1="19.05" y1="62.23" x2="17.78" y2="60.96" width="0.4064" layer="16"/>
 <wire x1="64.77" y1="37.465" x2="66.04" y2="36.195" width="0.4064" layer="1"/>
 <wire x1="64.77" y1="39.37" x2="64.77" y2="37.465" width="0.4064" layer="1"/>
@@
 <wire x1="66.04" y1="36.195" x2="66.04" y2="35.687" width="0.4064" layer="1"/>
 <wire x1="66.04" y1="40.64" x2="66.04" y2="40.767" width="0.4064" layer="1"/>
-<wire x1="59.69" y1="47.625" x2="59.69" y2="74.93" width="0.4064" layer="16"/>
+<wire x1="59.69" y1="47.625" x2="59.69" y2="67.2846" width="0.4064" layer="16"/>
+<wire x1="59.69" y1="67.2846" x2="59.69" y2="74.93" width="0.4064" layer="16"/>
 <wire x1="66.04" y1="41.275" x2="59.69" y2="47.625" width="0.4064" layer="16"/>
 <wire x1="66.04" y1="41.275" x2="66.04" y2="40.767" width="0.4064" layer="16"/>
@@
 <wire x1="24.765" y1="39.37" x2="24.13" y2="38.735" width="0.4064" layer="1"/>
 <wire x1="64.77" y1="39.37" x2="24.765" y2="39.37" width="0.4064" layer="1"/>
+<contactref element="J1" pad="40"/>
+<wire x1="24.13" y1="26.67" x2="25.4" y2="25.4" width="0.4064" layer="1"/>
+<wire x1="24.13" y1="38.1" x2="24.13" y2="26.67" width="0.4064" layer="1"/>
+<contactref element="JP6" pad="3"/>
+<contactref element="JP7" pad="1"/>
+<contactref element="JP7" pad="6"/>
+<wire x1="17.907" y1="61.0362" x2="19.05" y2="62.1792" width="0.4064" layer="16"/>
+<wire x1="19.05" y1="62.1792" x2="19.05" y2="62.23" width="0.4064" layer="16"/>
+<wire x1="17.907" y1="61.0362" x2="17.78" y2="60.96" width="0.4064" layer="16"/>
+<wire x1="39.3954" y1="55.3974" x2="39.3954" y2="54.6354" width="0.4064" layer="1"/>
+<wire x1="40.6146" y1="56.6166" x2="39.3954" y2="55.3974" width="0.4064" layer="1"/>
+<wire x1="40.6146" y1="66.0654" x2="40.6146" y2="56.6166" width="0.4064" layer="1"/>
+<wire x1="39.37" y1="67.31" x2="40.6146" y2="66.0654" width="0.4064" layer="1"/>
+<wire x1="39.3954" y1="54.6354" x2="39.37" y2="54.61" width="0.4064" layer="1"/>
+<wire x1="39.3954" y1="67.2846" x2="59.69" y2="67.2846" width="0.4064" layer="16"/>
+<wire x1="39.3954" y1="67.2846" x2="39.37" y2="67.31" width="0.4064" layer="16"/>
 </signal>
 <signal name="SDA">
 <contactref element="JP2" pad="4"/>
-<contactref element="JP3" pad="5"/>
 <contactref element="JP5" pad="5"/>
 <contactref element="J1" pad="3"/>
 <wire x1="17.78" y1="34.29" x2="19.05" y2="33.02" width="0.1524" layer="1"/>
 <wire x1="17.78" y1="55.88" x2="17.78" y2="34.29" width="0.1524" layer="1"/>
-<wire x1="19.05" y1="57.15" x2="17.78" y2="55.88" width="0.1524" layer="1"/>
 <wire x1="50.8" y1="71.12" x2="27.94" y2="71.12" width="0.1524" layer="16"/>
 <wire x1="54.61" y1="74.93" x2="50.8" y2="71.12" width="0.1524" layer="16"/>
-<wire x1="20.32" y1="58.42" x2="19.05" y2="57.15" width="0.1524" layer="1"/>
 <wire x1="20.32" y1="69.85" x2="20.32" y2="58.42" width="0.1524" layer="1"/>
 <wire x1="22.86" y1="72.39" x2="20.32" y2="69.85" width="0.1524" layer="1"/>
 <wire x1="27.94" y1="72.39" x2="22.86" y2="72.39" width="0.1524" layer="1"/>
 <wire x1="27.94" y1="71.12" x2="27.94" y2="72.39" width="0.1524" layer="1"/>
+<contactref element="JP6" pad="5"/>
+<wire x1="17.78" y1="55.88" x2="19.05" y2="57.15" width="0.1524" layer="1"/>
+<wire x1="20.32" y1="58.42" x2="19.05" y2="57.15" width="0.1524" layer="1"/>
 </signal>
 <signal name="SCL">
 <contactref element="JP2" pad="3"/>
-<contactref element="JP3" pad="4"/>
 <contactref element="JP5" pad="4"/>
 <contactref element="J1" pad="5"/>
 <wire x1="20.32" y1="36.83" x2="19.05" y2="35.56" width="0.1524" layer="16"/>
 <wire x1="20.32" y1="58.42" x2="20.32" y2="36.83" width="0.1524" layer="16"/>
-<wire x1="19.05" y1="59.69" x2="20.32" y2="58.42" width="0.1524" layer="16"/>
 <wire x1="50.8" y1="68.58" x2="32.385" y2="68.58" width="0.1524" layer="16"/>
 <wire x1="32.385" y1="68.58" x2="27.94" y2="68.58" width="0.1524" layer="16"/>
 <wire x1="57.15" y1="74.93" x2="50.8" y2="68.58" width="0.1524" layer="16"/>
-<wire x1="24.13" y1="64.77" x2="19.05" y2="59.69" width="0.1524" layer="16"/>
-<wire x1="28.575" y1="64.77" x2="24.13" y2="64.77" width="0.1524" layer="16"/>
-<wire x1="32.385" y1="68.58" x2="28.575" y2="64.77" width="0.1524" layer="16"/>
+<wire x1="32.385" y1="68.58" x2="28.956" y2="65.151" width="0.1524" layer="16"/>
+<contactref element="JP6" pad="4"/>
+<wire x1="20.2692" y1="58.4454" x2="19.05" y2="59.6646" width="0.1524" layer="16"/>
+<wire x1="19.05" y1="59.6646" x2="19.05" y2="59.69" width="0.1524" layer="16"/>
+<wire x1="20.2692" y1="58.4454" x2="20.32" y2="58.42" width="0.1524" layer="16"/>
+<wire x1="24.003" y1="58.4454" x2="20.3454" y2="58.4454" width="0.1524" layer="16"/>
+<wire x1="25.4508" y1="59.8932" x2="24.003" y2="58.4454" width="0.1524" layer="16"/>
+<wire x1="28.3464" y1="59.8932" x2="25.4508" y2="59.8932" width="0.1524" layer="16"/>
+<wire x1="28.956" y1="60.5028" x2="28.3464" y2="59.8932" width="0.1524" layer="16"/>
+<wire x1="28.956" y1="65.151" x2="28.956" y2="60.5028" width="0.1524" layer="16"/>
+<wire x1="20.3454" y1="58.4454" x2="20.32" y2="58.42" width="0.1524" layer="16"/>
 </signal>
 <signal name="INT">
@@
 <signal name="VCC1" class="2">
 <contactref element="JP2" pad="1"/>
-<contactref element="J1" pad="1"/>
-<wire x1="29.21" y1="72.39" x2="27.94" y2="73.66" width="0.3048" layer="1"/>
-<wire x1="29.21" y1="57.785" x2="29.21" y2="72.39" width="0.3048" layer="1"/>
+<wire x1="29.21" y1="57.785" x2="29.21" y2="58.42" width="0.3048" layer="1"/>
 <wire x1="28.575" y1="57.15" x2="29.21" y2="57.785" width="0.3048" layer="1"/>
 <wire x1="20.32" y1="57.15" x2="28.575" y2="57.15" width="0.3048" layer="1"/>
 <wire x1="20.32" y1="41.91" x2="20.32" y2="57.15" width="0.3048" layer="1"/>
 <wire x1="19.05" y1="40.64" x2="20.32" y2="41.91" width="0.3048" layer="1"/>
+<contactref element="J1" pad="13"/>
+<wire x1="29.21" y1="58.42" x2="27.94" y2="58.42" width="0.3048" layer="1"/>
 </signal>
 <signal name="THERM">
@@
 <contactref element="JP4" pad="2"/>
 </signal>
-<signal name="3.3V_GPS" class="2">
-<contactref element="JP3" pad="2"/>
-</signal>
-<signal name="VCC_GPS" class="1">
-<contactref element="JP3" pad="1"/>
-<contactref element="J1" pad="2"/>
-<wire x1="19.05" y1="67.31" x2="25.4" y2="73.66" width="0.4064" layer="16"/>
-</signal>
-<signal name="!RESET_GPS">
-<contactref element="JP3" pad="6"/>
-</signal>
 <signal name="3.3V_GYRO" class="2">
 <contactref element="JP5" pad="2"/>
@@
 <signal name="VCC_GYRO" class="1">
 <contactref element="JP5" pad="1"/>
-<contactref element="J1" pad="17"/>
-<wire x1="48.26" y1="73.66" x2="27.94" y2="53.34" width="0.4064" layer="1"/>
-<wire x1="64.77" y1="73.66" x2="48.26" y2="73.66" width="0.4064" layer="1"/>
+<wire x1="64.77" y1="73.66" x2="63.5" y2="73.66" width="0.4064" layer="1"/>
 <wire x1="64.77" y1="74.93" x2="64.77" y2="73.66" width="0.4064" layer="1"/>
+<contactref element="J1" pad="15"/>
+<wire x1="42.545" y1="52.705" x2="31.115" y2="52.705" width="0.4064" layer="1"/>
+<wire x1="27.94" y1="55.88" x2="31.115" y2="52.705" width="0.4064" layer="1"/>
+<wire x1="63.5" y1="73.66" x2="42.545" y2="52.705" width="0.4064" layer="1"/>
 </signal>
 <signal name="INT1">
@@
 <contactref element="JP5" pad="7"/>
 </signal>
+<signal name="VCC" class="1">
+<contactref element="JP6" pad="1"/>
+</signal>
+<signal name="1PPS">
+<contactref element="JP7" pad="2"/>
+</signal>
+<signal name="TXO">
+<contactref element="JP7" pad="5"/>
+</signal>
+<signal name="RXI">
+<contactref element="JP7" pad="4"/>
+</signal>
+<signal name="!RESET">
+<contactref element="JP6" pad="6"/>
+</signal>
+<signal name="N$1" class="2">
+<contactref element="JP6" pad="2"/>
+<contactref element="J1" pad="11"/>
+<wire x1="26.9748" y1="60.96" x2="27.94" y2="60.96" width="0.3048" layer="16"/>
+<wire x1="25.527" y1="62.4078" x2="26.9748" y2="60.96" width="0.3048" layer="16"/>
+<wire x1="21.4122" y1="62.4078" x2="25.527" y2="62.4078" width="0.3048" layer="16"/>
+<wire x1="19.05" y1="64.77" x2="21.4122" y2="62.4078" width="0.3048" layer="16"/>
+</signal>
 </signals>
